Commit message: created a urdf with calibration board

File: MotionPlanning/ur_description/urdf/ur5calibrate.urdf.xacro (robot description, xacro)
@@ -306,4 +306,37 @@
       <child link="${prefix}tool0"/>
     </joint>
+    <!--
+      ******************************
+      Not from the original urdf
+      ******************************
+      Adding calibration board here
+    -->
+    <link name="${prefix}calibrationboard">
+      <visual>
+        <geometry>
+          <box size="0.25 0.33 0.005">
+        </geometry>
+        <material name="LightGrey">
+          <color rgba="0.7 0.7 0.7 1.0"/>
+        </material>
+      </visual>
+      <collision>
+        <geometry>
+          <box size="0.25 0.33 0.005">
+        </geometry>
+      </collision>
+    </link>
+    <!-- Adding fixed link of calibration board here -->
+    <link name="${prefix}calibrationboard"/>
+    <joint name="${prefix}tool0-calibrationboard_fixed_joint" type="fixed">
+      <origin xyz="0 0 0.1" rpy="0 0 0"/>
+      <parent link="${prefix}tool0"/>
+      <child link="${prefix}calibrationboard"/>
+    </joint>
+     <!--
+      ******************************
+      This is the end of my edits
+      ******************************
+    -->
   </xacro:macro>
 </robot>

Commit message: added inertia

File: MotionPlanning/ur_description/urdf/ur5calibrate.urdf.xacro (robot description, xacro)
@@ -308,22 +308,25 @@
     <!--
       ******************************
-      Not from the original urdf
+      This is the start of edits
       ******************************
-      Adding calibration board here
     -->
     <link name="${prefix}calibrationboard">
       <visual>
         <geometry>
-          <box size="0.25 0.33 0.005">
-        </geometry>
-        <material name="LightGrey">
-          <color rgba="0.7 0.7 0.7 1.0"/>
-        </material>
-      </visual>
-      <collision>
-        <geometry>
-          <box size="0.25 0.33 0.005">
-        </geometry>
-      </collision>
+          <box size="0.25 0.33 0.005"/>
+        </geometry>
+        <material name="LightGrey">
+          <color rgba="0.7 0.7 0.7 1.0"/>
+        </material>
+      </visual>
+      <collision>
+        <geometry>
+          <box size="0.25 0.33 0.005"/>
+        </geometry>
+      </collision>
+      <inertial>
+         <mass value="0.3"/>
+         <inertia ixx="0.00273" ixy="0.0" ixz="0.0" iyy="0.00429" iyz="0.0" izz="0.00156"/>
+      </inertial>
     </link>
     <!-- Adding fixed link of calibration board here -->
